File: Hardware/InkTime.sch (EAGLE design)
At the start: 44 parts, among them IC1 BQ25180YBGR, IC2 BMA421, IC9 RT6160AWSC, U1 NRF52840_QF, X2 32.768kHz

Commit message: Add files via upload
Parts:
- added ANT1: 2450AT18B100E, InkTime_v5:2450AT18B100E_2450AT18B100E
- added C1, C2: 12pF, InkTime_v5:NORDIC_NRF_3_CAPACITOR_0201_L
- added C10, C22: N.C., InkTime_v5:NORDIC_NRF_3_CAPACITOR_0201_L
- added C11: 100pF, InkTime_v5:NORDIC_NRF_3_CAPACITOR_0201_L
- added C3, C4: 1pF, InkTime_v5:NORDIC_NRF_3_CAPACITOR_0201_L
- added C8: 100nF, InkTime_v5:NORDIC_NRF_3_CAPACITOR_0201_L
- added C9: 820pF, InkTime_v5:NORDIC_NRF_3_CAPACITOR_0201_L
- added J2: TC2030-IDC, InkTime_v5:TC2030-IDC_TC2030-IDC
- added L1: 3.9nH, InkTime_v5:NORDIC_NRF_2_INDUCTOR_0402_L
- added X1: 32MHz, InkTime_v5:NORDIC_NRF_XTAL_32MHZ
Connections:
- net N$40 renamed ALERT/2.5C
- net N$43 renamed P0.09
- net N$44 renamed P1.07
- net N$45 renamed P1.06
- net N$46 renamed P1.05
- net N$47 renamed P1.04
- net N$48 renamed P1.03
- net N$49 renamed P1.02/2.8C
- net N$50 renamed P1.01/2.4B
- new net N$40: C9.1, U1.DEC5@N24
- new net N$43: C11.1, U1.DEC3@D23
- new net N$44: C3.1, L1.1, U1.ANT@H23
- new net N$45: ANT1.FEED, C22.1, C4.1, L1.2
- new net N$46: C1.1, U1.XC1@B24, X1.1
- new net N$47: C2.1, U1.XC2@A23, X1.3
- new net N$48: J2.1
- new net N$49: J2.2
- new net N$50: J2.4
- new net N$54: J2.6
- net GND: now also C1.2, C10.2, C11.2, C2.2, C22.2, C3.2, C4.2, C8.2, C9.2, J2.3, J2.5, U1.VSS_PA@F23, U1.VSS_PAD, X1.2, X1.4
- net N$42: now also C10.1, U1.DEC6@E24
- net N$53: now also C8.1
Other:
- note added: "DEC3"
- note added: "N.C."
- note added: "RF"

Commit message: Add files via upload
Parts:
- added C1-EP-DR: 10uF, InkTime_v5:NORDIC_NRF_3_CAPACITOR_0201_L
- added C2-EP-DR: 4.7uF/25V, InkTime_v5:NORDIC_NRF_3_CAPACITOR_0201_L
- added C27, C34, C42: 0.1uF, InkTime_v5:GRM011R60J152KE01L_2_GRM011R60J152KE01L
- added C29, C30, C31, C32: 1uF, InkTime_v5:GRM011R60J152KE01L_2_GRM011R60J152KE01L
- added C43: 4.7μF, InkTime_v5:NORDIC_NRF_3_CAPACITOR_0201_L
- added D2, D4, D5: MBR0530, InkTime_v5:ESP32_C6_LIBRARY_5_MBR0530
- added D3: USBLC6-2SC6Y, InkTime_v5:ESP32_C6_LIBRARY_3_USBLC6-2SC6Y
- added EPD_C1, EPD_C10, EPD_C11, EPD_C12, EPD_C2, EPD_C6, EPD_C7, EPD_C8, EPD_C9: 1uF/50V, InkTime_v5:NORDIC_NRF_3_CAPACITOR_0201_L
- added EPD_C5: 0.1uF/50V, InkTime_v5:NORDIC_NRF_3_CAPACITOR_0201_L
- added IC3: BMA421, InkTime_v5:BMA423_BMA423
- added J1: 503480-2400, InkTime_v5:503480-2400_503480-2400
- added J4: KH-TYPE-C-16P, InkTime_v5:KH-TYPE-C-16P_KH-TYPE-C-16P
- added L5: 68uH, InkTime_v5:ESP32_C6_LIBRARY_2_744043680IND_4828-WE-TPC_WRE
- added Q1: 20V/4.2A/52mΩ/1.4W, InkTime_v5:ESP32_C6_LIBRARY_4_ESP32_WROVER_SPARKFUN-DISCRETESEMI_MOSFET_PCH-DMG2305UX-7
- added Q3: SI1308EDL-T1-GE3, InkTime_v5:ESP32_C6_LIBRARY_6_SI1308EDL-T1-GE3
- added R1_EP_DR: 0.47, InkTime_v5:ERA-1AEB3401C_CPF0201D7K68C1
- added R1_USB1, R2_USB: 5K1, InkTime_v5:ERA-1AEB3401C_CPF0201D7K68C1
- added R2_EP_DR, R5, R7, R8, R_PWR_EPD: 10K, InkTime_v5:ERA-1AEB3401C_CPF0201D7K68C1
- added R_TYPE_SEL: 2.2, InkTime_v5:ERA-1AEB3401C_CPF0201D7K68C1
- added SJ1: (no value), InkTime_v5:ESP32_C6_LIBRARY_7_JUMPER_SJ
- added SW_DN, SW_ENT, SW_UP: 2025-10-22_07-23-44_LIBRARY_EVP-AKE31ASW_EVP-AKE31A_PAN, InkTime_v5:2025-10-22_07-23-44_LIBRARY_EVP-AKE31ASW_EVP-AKE31A_PAN
- added TP_BAT_GND, TP_ON, TP_OP, TP_VBAT: HECTOR_WATCH_1_TPTP20R, InkTime_v5:HECTOR_WATCH_1_TPTP20R
- added U3: MAX17048G+T10, InkTime_v5:ESP32_C6_LIBRARY_MAX17048G+T10
- IC2: value BMA421 -> DRV2605YZFR; device InkTime_v5:BMA423_BMA423 -> InkTime_v5:DRV2605YZFR_DRV2605YZFR
Connections:
- removed net N$10: IC9.AGND, IC9.PGND_1, IC9.VSEL
- removed net N$11: TP_3V3.TP
- removed net N$12: TP_VREG.TP
- removed net N$16: C21.1, U1.VBUS@AD2
- removed net N$23: C6.1, U1.VDD@W1, U1.VDDH@Y2
- removed net N$25: TP_3.3V.TP
- removed net N$38: U1.P1.00@AD22
- removed net N$49: J2.2
- removed net N$50: J2.4
- removed net N$51: U1.SWDIO@AC24
- removed net N$52: U1.SWDCLK@AA24
- removed net N$54: J2.6
- new net 3V3/1.7D: R5.2, R7.2, R8.2
- new net ALERT/1.6C: U3.!ALERT
- new net D+/1.5D: D3.I/O2_2
- new net D-/1.5D: D3.I/O1_2
- new net DN: J4.DN1
- new net DP: J4.DP1
- new net EPD_3V3: EPD_C5.2, J1.15, J1.16
- new net EPD_BUSY/1.5D: J1.9
- new net EPD_CS/1.4C: J1.12
- new net EPD_DC/1.5D: J1.11
- new net EPD_RST/1.5D: J1.10
- new net GDR: J1.2
- new net HAPTIC_EN/1.4C: IC2.EN
- new net MOSI/1.5B: J1.14
- new net N$55: EPD_C1.2, J1.5
- new net N$56: EPD_C2.2, J1.4
- new net N$57: EPD_C6.2, J1.18
- new net N$58: EPD_C7.2, J1.19
- new net N$59: EPD_C9.2, J1.21
- new net N$60: EPD_C8.2, J1.20
- new net N$61: EPD_C10.2, J1.22
- new net N$62: EPD_C11.2, J1.23
- new net N$63: EPD_C12.2, J1.24
- new net N$64: J4.DN2
- new net N$65: J4.DP2
- new net N$66: J4.CC1, R1_USB1.2
- new net N$67: J4.CC2, R2_USB.1
- new net N$68: C42.1, C43.1
- new net N$70: D3.VBUS
- new net N$71: C32.2, IC2.REG
- new net N$72: D3.I/O1_1
- new net N$74: D3.I/O2_1
- new net N$77: Q1.S
- new net N$78: C34.2, IC2.VDD
- new net N$80: R_PWR_EPD.2
- new net N$81: Q1.D
- new net N$82: Q3.G, R2_EP_DR.2
- new net N$83: Q3.S, R1_EP_DR.2
- new net N$84: R1_EP_DR.1, R_TYPE_SEL.2, SJ1.2
- new net N$85: C2-EP-DR.1, D5.A, L5.1, Q3.D
- new net N$86: C2-EP-DR.2, D2.K, D4.A
- new net N$87: C1-EP-DR.2, L5.2
- new net OUT+: IC2.OUT+, TP_OP.TP
- new net OUT-: IC2.OUT-, TP_ON.TP
- new net P0.13/1.5D: C30.2, R5.1, SW_UP.2
- new net P0.14/1.5D: C31.2, R8.1, SW_ENT.2
- new net P1.01/1.6C: Q1.G, R_PWR_EPD.1
- new net P1.02/1.6C: C29.2, R7.1, SW_DN.2
- new net PREVGH: D5.K
- new net PREVGL: D2.A
- new net RESE: J1.3
- new net SCK/1.5B: J1.13
- new net SCL/1.4C: IC2.SCL, U3.SCL
- new net SDA/1.4C: IC2.SDA, U3.SDA
- new net VBAT/1.2A: C27.2, TP_VBAT.TP, U3.CELL, U3.VDD
- new net VBUS/1.5D: J4.VBUS
- net 3V3/2.4A: now also C6.1, TP_3.3V.TP, TP_3V3.TP, U1.VDD@W1, U1.VDDH@Y2
- net GND: now also C1-EP-DR.1, C27.1, C29.1, C30.1, C31.1, C32.1, C34.1, C42.2, C43.2, D3.GND, D4.K, EPD_C1.1, EPD_C10.1, EPD_C11.1, EPD_C12.1, EPD_C2.1, EPD_C5.1, EPD_C6.1, EPD_C7.1, EPD_C8.1, EPD_C9.1, IC2.IN/TRIG, IC3.GND, IC3.GNDIO, IC9.AGND, IC9.PGND_1, IC9.VSEL, J1.17, J1.8, J1.MP1, J1.MP2, J4.GND, J4.SHIELD, R1_USB1.1, R2_EP_DR.1, R2_USB.2, R_TYPE_SEL.1, SJ1.1, SW_DN.1, SW_ENT.1, SW_UP.1, TP_BAT_GND.TP, U3.CTG, U3.EP, U3.GND, U3.QSTRT; no longer IC2.GNDIO
- net IMU_INT1: now also IC3.INT1; no longer IC2.INT1
- net IMU_INT2: now also IC3.INT2; no longer IC2.INT2
- net N$18: now also IC3.CSB, IC3.VDD; no longer IC2.CSB, IC2.VDD
- net N$19: now also IC3.SCX; no longer IC2.SCX
- net N$20: now also IC3.VDDIO; no longer IC2.VDDIO
- net N$21: now also IC3.SDX; no longer IC2.SDX
- net N$22: now also IC3.SDO; no longer IC2.SDO
- net RESET: now also J2.6
- net SWDCLK: now also J2.4, U1.SWDCLK@AA24
- net SWDIO: now also J2.2, U1.SWDIO@AC24
- net SWO: now also U1.P1.00@AD22
- net VBUS/2.6D: now also C21.1, U1.VBUS@AD2
- net VREG: now also TP_VREG.TP
Other:
- note added: "Buttons"
- note added: "DMG2305UX-7"
- note added: "Driver"
- note added: "E-Paper & Peripherals"
- note added: "E-Paper Display Connector"
- note added: "E-Paper Drive Circuit"
- note added: "Fuel Gauge"
- note added: "Haptic"
- note added: "MCU, Power, IMU, SWD"
- note added: "Protection"
- note added: "USB C Connector & ESD"
- note added: "drawn by: Cebotari Nichita"
